File: Smart_switch_edge_AI_V2.brd (EAGLE design)
At the start: 60.6 x 40.8 mm, 13 parts, among them K1 AQG12105, K2 AQG12105, K3 AQG12105

Commit message: Add files via upload
Parts:
- moved K1 2.00 mm to (1.81, 19.1), flipped to the bottom
- moved K3 1.40 mm to (58.5, 19.1), flipped to the bottom
- moved K2 0.79 mm to (31.1, 4.09), flipped to the bottom, turned to 180 degrees
- flipped U$2 to the bottom, turned to 270 degrees
- flipped X1 to the bottom
- flipped X2 to the bottom
Routing:
- net N$10: track 149.3 -> 115.7 mm, vias 5 -> 4
- net N$5: track 54.5 -> 37.2 mm, vias 2 -> 0
- net GND: track 152.0 -> 134.9 mm
- net N$9: track 12.8 -> 25.4 mm, vias 3 -> 0
- net +5V: track 45.7 -> 39.3 mm
- net N$7: track 58.1 -> 64.2 mm, vias 3 -> 0
- net N$11: track 29.2 -> 34.7 mm
- net N$3: track 29.6 -> 33.9 mm, vias 0 -> 2
- net N$6: track 96.6 -> 93.6 mm, vias 0 -> 2
- net N$4: track 20.0 -> 22.0 mm
- net N$2: track 37.6 -> 39.3 mm, vias 0 -> 2
- net N$8: track 22.3 -> 21.1 mm, vias 2 -> 3
- net N$1: vias 0 -> 2

Commit message: Add files via upload
Parts:
- added JP1, JP2, JP3, JP4, JP5, JP6: (no value), adafruit:1X1-BIGPOGO
- moved K1 0.45 mm to (2.01, 19.4)
- moved K3 0.30 mm to (58.5, 19.4)
Connections:
- new net N$12: JP2.P$1, U$1.18
- new net N$13: JP3.P$1, U$1.17
- net +5V: now also JP1.P$1
- net GND: now also JP4.P$1
- net N$1: now also JP6.P$1
- net N$2: now also JP5.P$1
Routing:
- net N$2: track 39.3 -> 107.1 mm, vias 2 -> 4
- net N$1: track 19.3 -> 82.0 mm, vias 2 -> 5
- net +5V: track 39.3 -> 67.9 mm
- net N$12: track 0.00 -> 10.5 mm, vias 0 -> 1
- net N$13: track 0.00 -> 10.5 mm, vias 0 -> 1
- net N$10: track 115.7 -> 111.3 mm
- net N$4: track 22.0 -> 21.4 mm
