File: Smart_switch_edge_AI_V2.sch (EAGLE design)
At the start: 13 parts, among them K1 AQG12105, K2 AQG12105, K3 AQG12105

Commit message: Add files via upload
Parts:
- added JP1, JP2, JP3, JP4, JP5, JP6: (no value), adafruit:PINHD-1X1-BIGPOGO
Connections:
- new net N$12: JP2.1, U$1.TX
- new net N$13: JP3.1, U$1.RX
- net +5V: now also JP1.1
- net GND: now also JP4.1
- net N$1: now also JP6.1
- net N$2: now also JP5.1
